File: cabinetLed.kicad_pcb (KiCad board)
At the start: 2 copper layers, 31 parts, among them U1 MDBT42V-512KV2, U2 BQ25185, U3 MIC5504-3.3YM5, Y1 DST410S

Commit message: 2024-02-22_2
Parts:
- U3: moved to B.Cu
- moved U3 33.2 mm to (144.1, 70.6)
Changed lines of the file:
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@@
-    )
-  )
-  (footprint "Package_TO_SOT_SMD:SOT-23-5" (layer "F.Cu")
-    (at 111.577 64.027)
-    (descr "SOT, 5 Pin (https://www.jedec.org/sites/default/files/docs/Mo-178c.PDF variant AA), generated with kicad-footprint-generator ipc_gullwing_generator.py")
-    (tags "SOT TO_SOT_SMD")
-    (property "Sheetfile" "cabinetLed.kicad_sch")
-    (property "Sheetname" "")
-    (property "ki_description" "300mA Low-dropout Voltage Regulator, Vout 3.3V, Vin up to 5.5V, SOT-23")
-    (property "ki_keywords" "Micrel LDO voltage regulator")
-    (attr smd)
-    (fp_text reference "U3" (at 0 -2.4) (layer "F.SilkS")
-        (effects (font (size 1 1) (thickness 0.15)))
-    )
-    (fp_text value "MIC5504-3.3YM5" (at 0 2.4) (layer "F.Fab")
-        (effects (font (size 1 1) (thickness 0.15)))
-    )
-    (fp_text user "${REFERENCE}" (at 0 0) (layer "F.Fab")
-        (effects (font (size 0.4 0.4) (thickness 0.06)))
-    )
-    (fp_line (start 0 -1.56) (end -1.8 -1.56)
-      (stroke (width 0.12) (type solid)) (layer "F.SilkS"))
-    (fp_line (start 0 -1.56) (end 0.8 -1.56)
-      (stroke (width 0.12) (type solid)) (layer "F.SilkS"))
-    (fp_line (start 0 1.56) (end -0.8 1.56)
-      (stroke (width 0.12) (type solid)) (layer "F.SilkS"))
-    (fp_line (start 0 1.56) (end 0.8 1.56)
-      (stroke (width 0.12) (type solid)) (layer "F.SilkS"))
-    (fp_line (start -2.05 -1.7) (end -2.05 1.7)
-      (stroke (width 0.05) (type solid)) (layer "F.CrtYd"))
-    (fp_line (start -2.05 1.7) (end 2.05 1.7)
-      (stroke (width 0.05) (type solid)) (layer "F.CrtYd"))
-    (fp_line (start 2.05 -1.7) (end -2.05 -1.7)
-      (stroke (width 0.05) (type solid)) (layer "F.CrtYd"))
-    (fp_line (start 2.05 1.7) (end 2.05 -1.7)
-      (stroke (width 0.05) (type solid)) (layer "F.CrtYd"))
-    (fp_line (start -0.8 -1.05) (end -0.4 -1.45)
-      (stroke (width 0.1) (type solid)) (layer "F.Fab"))
-    (fp_line (start -0.8 1.45) (end -0.8 -1.05)
-      (stroke (width 0.1) (type solid)) (layer "F.Fab"))
-    (fp_line (start -0.4 -1.45) (end 0.8 -1.45)
-      (stroke (width 0.1) (type solid)) (layer "F.Fab"))
-    (fp_line (start 0.8 -1.45) (end 0.8 1.45)
-      (stroke (width 0.1) (type solid)) (layer "F.Fab"))
-    (fp_line (start 0.8 1.45) (end -0.8 1.45)
-      (stroke (width 0.1) (type solid)) (layer "F.Fab"))
-    (pad "1" smd roundrect (at -1.1375 -0.95) (size 1.325 0.6) (layers "F.Cu" "F.Paste" "F.Mask") (roundrect_rratio 0.25)
-      (net 4 "VDD") (pinfunction "VIN") (pintype "power_in"))
-    (pad "2" smd roundrect (at -1.1375 0) (size 1.325 0.6) (layers "F.Cu" "F.Paste" "F.Mask") (roundrect_rratio 0.25)
-      (net 2 "GND") (pinfunction "GND") (pintype "power_in"))
-    (pad "3" smd roundrect (at -1.1375 0.95) (size 1.325 0.6) (layers "F.Cu" "F.Paste" "F.Mask") (roundrect_rratio 0.25)
-      (net 26 "Net-(U3-EN)") (pinfunction "EN") (pintype "input"))
-    (pad "4" smd roundrect (at 1.1375 0.95) (size 1.325 0.6) (layers "F.Cu" "F.Paste" "F.Mask") (roundrect_rratio 0.25)
-      (net 41 "unconnected-(U3-NC-Pad4)") (pinfunction "NC") (pintype "no_connect"))
-    (pad "5" smd roundrect (at 1.1375 -0.95) (size 1.325 0.6) (layers "F.Cu" "F.Paste" "F.Mask") (roundrect_rratio 0.25)
-      (net 6 "+3V3") (pinfunction "VOUT") (pintype "power_out"))
-    (model "${KICAD6_3DMODEL_DIR}/Package_TO_SOT_SMD.3dshapes/SOT-23-5.wrl"
-      (offset (xyz 0 0 0))
-      (scale (xyz 1 1 1))
-      (rotate (xyz 0 0 0))
     )
   )
@@
       (offset (xyz 0 0 0))
       (scale (xyz 1 1 1))
+      (rotate (xyz 0 0 0))
+    )
+  )
+  (footprint "Package_TO_SOT_SMD:SOT-23-5" (layer "B.Cu")
+    (at 144.145 70.612)
+    (descr "SOT, 5 Pin (https://www.jedec.org/sites/default/files/docs/Mo-178c.PDF variant AA), generated with kicad-footprint-generator ipc_gullwing_generator.py")
+    (tags "SOT TO_SOT_SMD")
+    (property "Sheetfile" "cabinetLed.kicad_sch")
+    (property "Sheetname" "")
+    (property "ki_description" "300mA Low-dropout Voltage Regulator, Vout 3.3V, Vin up to 5.5V, SOT-23")
+    (property "ki_keywords" "Micrel LDO voltage regulator")
+    (attr smd)
+    (fp_text reference "U3" (at 0 2.4) (layer "B.SilkS")
+        (effects (font (size 1 1) (thickness 0.15)) (justify mirror))
+    )
+    (fp_text value "MIC5504-3.3YM5" (at 0 -2.4) (layer "B.Fab")
+        (effects (font (size 1 1) (thickness 0.15)) (justify mirror))
+    )
+    (fp_text user "${REFERENCE}" (at 0 0) (layer "B.Fab")
+        (effects (font (size 0.4 0.4) (thickness 0.06)) (justify mirror))
+    )
+    (fp_line (start 0 -1.56) (end -0.8 -1.56)
+      (stroke (width 0.12) (type solid)) (layer "B.SilkS"))
+    (fp_line (start 0 -1.56) (end 0.8 -1.56)
+      (stroke (width 0.12) (type solid)) (layer "B.SilkS"))
+    (fp_line (start 0 1.56) (end -1.8 1.56)
+      (stroke (width 0.12) (type solid)) (layer "B.SilkS"))
+    (fp_line (start 0 1.56) (end 0.8 1.56)
+      (stroke (width 0.12) (type solid)) (layer "B.SilkS"))
+    (fp_line (start -2.05 -1.7) (end 2.05 -1.7)
+      (stroke (width 0.05) (type solid)) (layer "B.CrtYd"))
+    (fp_line (start -2.05 1.7) (end -2.05 -1.7)
+      (stroke (width 0.05) (type solid)) (layer "B.CrtYd"))
+    (fp_line (start 2.05 -1.7) (end 2.05 1.7)
+      (stroke (width 0.05) (type solid)) (layer "B.CrtYd"))
+    (fp_line (start 2.05 1.7) (end -2.05 1.7)
+      (stroke (width 0.05) (type solid)) (layer "B.CrtYd"))
+    (fp_line (start -0.8 -1.45) (end -0.8 1.05)
+      (stroke (width 0.1) (type solid)) (layer "B.Fab"))
+    (fp_line (start -0.8 1.05) (end -0.4 1.45)
+      (stroke (width 0.1) (type solid)) (layer "B.Fab"))
+    (fp_line (start -0.4 1.45) (end 0.8 1.45)
+      (stroke (width 0.1) (type solid)) (layer "B.Fab"))
+    (fp_line (start 0.8 -1.45) (end -0.8 -1.45)
+      (stroke (width 0.1) (type solid)) (layer "B.Fab"))
+    (fp_line (start 0.8 1.45) (end 0.8 -1.45)
+      (stroke (width 0.1) (type solid)) (layer "B.Fab"))
+    (pad "1" smd roundrect (at -1.1375 0.95) (size 1.325 0.6) (layers "B.Cu" "B.Paste" "B.Mask") (roundrect_rratio 0.25)
+      (net 4 "VDD") (pinfunction "VIN") (pintype "power_in"))
+    (pad "2" smd roundrect (at -1.1375 0) (size 1.325 0.6) (layers "B.Cu" "B.Paste" "B.Mask") (roundrect_rratio 0.25)
+      (net 2 "GND") (pinfunction "GND") (pintype "power_in"))
+    (pad "3" smd roundrect (at -1.1375 -0.95) (size 1.325 0.6) (layers "B.Cu" "B.Paste" "B.Mask") (roundrect_rratio 0.25)
+      (net 26 "Net-(U3-EN)") (pinfunction "EN") (pintype "input"))
+    (pad "4" smd roundrect (at 1.1375 -0.95) (size 1.325 0.6) (layers "B.Cu" "B.Paste" "B.Mask") (roundrect_rratio 0.25)
+      (net 41 "unconnected-(U3-NC-Pad4)") (pinfunction "NC") (pintype "no_connect"))
+    (pad "5" smd roundrect (at 1.1375 0.95) (size 1.325 0.6) (layers "B.Cu" "B.Paste" "B.Mask") (roundrect_rratio 0.25)
+      (net 6 "+3V3") (pinfunction "VOUT") (pintype "power_out"))
+    (model "${KICAD6_3DMODEL_DIR}/Package_TO_SOT_SMD.3dshapes/SOT-23-5.wrl"
+      (offset (xyz 0 0 0))
+      (scale (xyz 1 1 1))
