File: cabinetLed.kicad_sch (KiCad schematic)
At the start: 31 parts, among them U1 MDBT42V-512KV2, U2 BQ25185, U3 MIC5504-3.3YM5, Y1 DST410S

Commit message: 2024-02-22_2
Parts:
- removed U2: BQ25185, Library:WSON-10-1EP_2.1x2.1mm_P0.4mm_EP0.9x1.5mm, symbol New_Library:BQ25185
- removed U3: MIC5504-3.3YM5, Package_TO_SOT_SMD:SOT-23-5, symbol Regulator_Linear:MIC5504-3.3YM5
- added C10: 4.7uF/1005, Capacitor_SMD:C_0402_1005Metric, symbol Device:C_Small
- added C11: 10pF/1005, Capacitor_SMD:C_0402_1005Metric, symbol Device:C_Small
- added C12: 10uF/1005, Capacitor_SMD:C_0402_1005Metric, symbol Device:C_Small
- added L3: 10uH/1608, symbol Device:L_Small
- added U4: LTC3553, Package_DFN_QFN:QFN-20-1EP_3x3mm_P0.4mm_EP1.65x1.65mm, symbol Battery_Management:LTC3553
- C2: value 1uF/1005 -> 10uF/1005
- R1: value 1K/1005 -> 649K/1005; footprint Resistor_SMD:R_0402_1005Metric -> (none)
- R2: value 5K/1005 -> 649K/1005; footprint Resistor_SMD:R_0402_1005Metric -> (none)
- R3, R4: value 10K/1005 -> 649K/1005; footprint Resistor_SMD:R_0402_1005Metric -> (none)
Connections:
- net +3V3: now also R1.2, R3.2, C10.1, C11.1, C12.1, L3.2, U4.10 (LDO)
- net GND: now also C2.1, C10.2, U4.15 (NTC), U4.2 (SEQ), U4.21 (GND); no longer C2.2, R1.2, R3.2
- net at R2.1: now also R1.1, U4.9 (LDO_FB)
- net at R4.2: now also C12.2
- net at H2.1: now also U4.17 (BAT); no longer C4.1
- net at H1.1: now also C2.2, U4.20 (VBUS); no longer C2.1
- net at R3.1: now also R4.1, C11.2, U4.8 (BUCK_FB)
- removed net VDD: C3.1, C5.1, R4.1
- new net: U4.11 (VINLDO), U4.12 (BVIN)
- new net: L3.1, U4.13 (SW)
- no-connect marks 9 -> 10
Other:
- moved on the sheet: C2, C6, H1, H2

Commit message: 2024-02-23
Parts:
- removed C3: 10uF/1005, Capacitor_SMD:C_0402_1005Metric, symbol Device:C_Small
- removed C4: 1uF/1005, Capacitor_SMD:C_0402_1005Metric, symbol Device:C_Small
Changed lines of the file:
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@@
   (junction (at 78.74 162.56) (diameter 0) (color 0 0 0 0)
-  )
-  (junction (at 43.18 66.04) (diameter 0) (color 0 0 0 0)
   )
   (junction (at 224.79 73.66) (diameter 0) (color 0 0 0 0)
@@
     (stroke (width 0) (type default))
   )
-  (wire (pts (xy 43.18 52.07) (xy 43.18 57.15))
-    (stroke (width 0) (type default))
-  )
   (wire (pts (xy 104.14 99.06) (xy 104.14 101.6))
     (stroke (width 0) (type default))
@@
     (stroke (width 0) (type default))
   )
+  (wire (pts (xy 50.8 68.58) (xy 58.42 68.58))
+    (stroke (width 0) (type default))
+  )
   (wire (pts (xy 162.56 71.12) (xy 170.18 71.12))
     (stroke (width 0) (type default))
@@
     (stroke (width 0) (type default))
   )
+  (wire (pts (xy 50.8 66.04) (xy 58.42 66.04))
+    (stroke (width 0) (type default))
+  )
   (wire (pts (xy 203.2 68.58) (xy 203.2 76.2))
     (stroke (width 0) (type default))
@@
     (stroke (width 0) (type default))
   )
+  (wire (pts (xy 50.8 73.66) (xy 58.42 73.66))
+    (stroke (width 0) (type default))
+  )
   (wire (pts (xy 251.46 72.39) (xy 247.65 72.39))
     (stroke (width 0) (type default))
@@
     (stroke (width 0) (type default))
   )
-  (wire (pts (xy 43.18 62.23) (xy 43.18 66.04))
-    (stroke (width 0) (type default))
-  )
   (wire (pts (xy 99.06 101.6) (xy 99.06 109.22))
     (stroke (width 0) (type default))
@@
     (stroke (width 0) (type default))
   )
+  (wire (pts (xy 50.8 78.74) (xy 58.42 78.74))
+    (stroke (width 0) (type default))
+  )
   (wire (pts (xy 166.37 60.96) (xy 170.18 60.96))
     (stroke (width 0) (type default))
@@
     (stroke (width 0) (type default))
   )
-  (wire (pts (xy 43.18 66.04) (xy 49.53 66.04))
-    (stroke (width 0) (type default))
-  )
   (wire (pts (xy 200.66 55.88) (xy 209.55 55.88))
     (stroke (width 0) (type default))
@@
     (stroke (width 0) (type default))
   )
+  (wire (pts (xy 50.8 76.2) (xy 58.42 76.2))
+    (stroke (width 0) (type default))
+  )
   (wire (pts (xy 78.74 162.56) (xy 85.09 162.56))
     (stroke (width 0) (type default))
@@
     (stroke (width 0) (type default))
   )
-  (wire (pts (xy 43.18 66.04) (xy 43.18 71.12))
-    (stroke (width 0) (type default))
-  )
   (wire (pts (xy 64.77 165.1) (xy 73.66 165.1))
     (stroke (width 0) (type default))
@@
   )
   (wire (pts (xy 104.14 82.55) (xy 104.14 85.09))
-    (stroke (width 0) (type default))
-  )
-  (wire (pts (xy 49.53 64.77) (xy 49.53 66.04))
     (stroke (width 0) (type default))
   )
@@
     )
   )
-  (symbol (lib_id "Device:C_Small") (at 43.18 59.69 0) (mirror y) (unit 1)
-    (in_bom yes) (on_board yes) (dnp no)
-    (property "Reference" "C3" (at 40.64 58.42 0)
-      (effects (font (size 1.27 1.27)) (justify left))
-    )
-    (property "Value" "10uF/1005" (at 40.64 60.96 0)
-      (effects (font (size 1.27 1.27)) (justify left))
-    )
-    (property "Footprint" "Capacitor_SMD:C_0402_1005Metric" (at 43.18 59.69 0)
-      (effects (font (size 1.27 1.27)) hide)
-    )
-    (property "Datasheet" "~" (at 43.18 59.69 0)
-      (effects (font (size 1.27 1.27)) hide)
-    )
-    (pin "2")
-    (pin "1")
-    (instances
-      (project "cabinetLed"
-        (path "/d628c071-57e2-4deb-8227-483fbff81687"
-          (reference "C3") (unit 1)
-        )
-      )
-    )
-  )
   (symbol (lib_id "Device:R_Small_US") (at 38.1 160.02 90) (unit 1)
     (in_bom yes) (on_board yes) (dnp no)
@@
     )
   )
-  (symbol (lib_id "Device:C_Small") (at 49.53 62.23 0) (mirror y) (unit 1)
-    (in_bom yes) (on_board yes) (dnp no)
-    (property "Reference" "C4" (at 46.99 60.96 0)
-      (effects (font (size 1.27 1.27)) (justify left))
-    )
-    (property "Value" "1uF/1005" (at 46.99 63.5 0)
-      (effects (font (size 1.27 1.27)) (justify left))
-    )
-    (property "Footprint" "Capacitor_SMD:C_0402_1005Metric" (at 49.53 62.23 0)
-      (effects (font (size 1.27 1.27)) hide)
-    )
-    (property "Datasheet" "~" (at 49.53 62.23 0)
-      (effects (font (size 1.27 1.27)) hide)
-    )
-    (pin "2")
-    (pin "1")
-    (instances
-      (project "cabinetLed"
-        (path "/d628c071-57e2-4deb-8227-483fbff81687"
-          (reference "C4") (unit 1)
-        )
-      )
-    )
-  )
   (symbol (lib_id "Device:C_Small") (at 203.2 80.01 0) (unit 1)
     (in_bom yes) (on_board yes) (dnp no) (fields_autoplaced)
@@
         )
       )
-    )
-  )
-  (symbol (lib_id "power:GND") (at 43.18 71.12 0) (unit 1)
-    (in_bom yes) (on_board yes) (dnp no) (fields_autoplaced)
-    (property "Reference" "#PWR09" (at 43.18 77.47 0)
-      (effects (font (size 1.27 1.27)) hide)
-    )
-    (property "Value" "GND" (at 43.18 76.2 0)
-      (effects (font (size 1.27 1.27)) hide)
-    )
-    (property "Footprint" "" (at 43.18 71.12 0)
-      (effects (font (size 1.27 1.27)) hide)
-    )
-    (property "Datasheet" "" (at 43.18 71.12 0)
-      (effects (font (size 1.27 1.27)) hide)
-    )
-    (pin "1")
-    (instances
-      (project "cabinetLed"
-        (path "/d628c071-57e2-4deb-8227-483fbff81687"
-          (reference "#PWR09") (unit 1)
-        )
-      )

Commit message: 2024-02-26 change led
Parts:
- removed C5, C6: 1uF/1005, Capacitor_SMD:C_0402_1005Metric, symbol Device:C_Small
- removed D1, D2: ASMT-YTB7-0AA02, LED_SMD:LED_Avago_PLCC6_3x2.8mm, symbol LED:ASMT-YTB7-0AA02
- removed R10, R7, R9: 3/1608, Resistor_SMD:R_0603_1608Metric, symbol Device:R_Small_US
- removed R6: 3/1608, Resistor_SMD:R_0402_1005Metric, symbol Device:R_Small_US
- removed R8: 24/1608, Resistor_SMD:R_0603_1608Metric, symbol Device:R_Small_US
- added C3, C4: 100nF/1005, Capacitor_SMD:C_0402_1005Metric, symbol Device:C_Small
- added LED1, LED2: WS2812B-2020, symbol New_Library:WS2812B-2020
- R5: value 24/1608 -> 649K/1005; footprint Resistor_SMD:R_0603_1608Metric -> (none)
Connections:
- net +3V3: no longer C11.1, C12.1, L3.2, R3.2, R5.1
- net GND: now also C12.2, R4.2, R5.1, C3.2, C4.2, LED1.2 (GND), LED2.2 (GND)
- net at R5.2: now also U4.16 (PROG)
- net B_BLUE: no longer names the net of U1.26 (P0.02)
- net B_GREEN: no longer names the net of U1.27 (P0.03)
- net B_RED renamed DI
- net DI: now also LED1.3 (DI)
- net H_BLUE: no longer names the net of U1.11 (P0.09)
- net H_GREEN: no longer names the net of U1.12 (P0.08)
- net H_RED: no longer names the net of U1.13 (P0.10)
- new net: LED1.1 (DO), LED2.3 (DI)
- new net +5V: C11.1, C12.1, C3.1, C4.1, L3.2, LED1.4 (VDD), LED2.4 (VDD), R3.2
- no-connect marks 10 -> 16
Other:
- note added: "ICHG(A) = 750V/RPROG"
- moved on the sheet: C10, C11, C12, C2, H1, H2, L3, R1, R2, R3, R4, U4

Commit message: 2024-02-28
Parts:
- removed H1: VIN_Pad, MountingHole:MountingHole_2.2mm_M2, symbol Mechanical:MountingHole_Pad
- removed H2: BAT_Pad, MountingHole:MountingHole_2.2mm_M2, symbol Mechanical:MountingHole_Pad
- removed U4: LTC3553, Package_DFN_QFN:QFN-20-1EP_3x3mm_P0.4mm_EP1.65x1.65mm, symbol Battery_Management:LTC3553
- added C13, C15, C6: 1uF/1005, Capacitor_SMD:C_0402_1005Metric, symbol Device:C_Small
- added C14: 2.2uF/1005, Capacitor_SMD:C_0402_1005Metric, symbol Device:C_Small
- added C5: 4.7uF/1005, Capacitor_SMD:C_0402_1005Metric, symbol Device:C_Small
- added L4: 4.7uH/1608, symbol Device:L_Small
- added TP3: TestPoint_BAT, TestPoint:TestPoint_Pad_D2.0mm, symbol Connector:TestPoint
- added U2: ADP5350, symbol New_Library:ADP5350
- C10: value 4.7uF/1005 -> 10uF/1005
- C11: value 10pF/1005 -> 10uF/1005
- C12: value 10uF/1005 -> 4.7uF/1005
- L3: value 10uH/1608 -> 1.5uH/1608
- R1, R2: value 649K/1005 -> R_Small_US
- R3, R4: value 649K/1005 -> 10K/1608
- R5: value 649K/1005 -> 47K/1608
Connections:
- net +3V3: now also C15.1, U2.29 (VOUT1); no longer C10.1, R1.2
- net +5V: now also R1.1, U2.17 (VOUT4); no longer C11.1, C12.1, L3.2, R3.2
- net DI: now also U1.11 (P0.09)
- net GND: now also C11.2, C2.2, C13.2, C14.2, C15.2, C5.2, C6.2, U2.10 (PGND1B), U2.16 (PGND4), U2.33 (EP), U2.9 (PGND1A); no longer C2.1, R4.2, R5.1
- net at R5.2: now also U2.3 (THR)
- net at R3.1, R4.1: no longer C11.2
- net SCL: now reaches U1.5 (P0.20)
- net SCL: now also R3.2, U2.30 (SCL)
- net PGOOD: now reaches U1.9 (P0.12)
- net PGOOD: now also U2.2 (PGOOD)
- net VSYS: now reaches L3.1
- net VSYS: now also C10.1, C12.1, C13.1, C6.1, L4.2, U2.19 (VIN4), U2.27 (VIN123), U2.6 (ISOS)
- net at R2.1: now also R1.2, U2.18 (FB4); no longer R1.1
- net STAT1 renamed SDA
- net SDA: now also R4.2, U2.31 (SDA)
- net STAT2 renamed BATOK
- net BATOK: now also U2.32 (BATOK)
- net /CE renamed ~{INT}
- net ~{INT}: now also U2.1 (~{INT})
- new net: L3.2, U2.11 (SW1A), U2.12 (SW1B)
- new net: L4.1, U2.15 (SW4)
- new net: C14.1, U2.26 (CFL2)
- new net: C11.1, TP3.1, U2.4 (BSNS), U2.5 (ISOB)
- new net: C5.1, U2.8 (CFL1)
- new net GNDA: R5.1, U2.7 (AGND)
- new net VCC: C2.1, U2.13 (VBUSA), U2.14 (VBUSB)
Other:
- note removed: "ICHG(A) = 750V/RPROG"
